File: FW_RP-2040_Probe/FW_RP-2040_Probe.kicad_sch (KiCad schematic)
At the start: 38 parts, among them P1 USB_C_Plug_USB2.0, P2 JST Female 1x3, P3 JST Female 1x3, U1 AP2112K-3.3, U2 RP2040, U3 W25Q128JVS, U4 MC74VHC1GT126, U5 MC74VHC1GT126, Y1 RH100-12.000-9-1015-TR-NS1

Commit message: Update schematic to pinout v1.1.1, update layout to v0.5.0
Parts:
- removed C10: 10nF, Capacitor_SMD:C_0402_1005Metric, symbol Device:C_Small
- added TP4, TP5: TestPoint, KKicadLib:TestPoint_Pad_1.5x1.5mm_THT, symbol Connector:TestPoint
- DB1, DB2, DB3, TP1, TP2, TP3: footprint TestPoint:TestPoint_Pad_1.5x1.5mm -> KKicadLib:TestPoint_Pad_1.5x1.5mm_THT
- renumbered U5 to U4, U4 to U5
Connections:
- net +1V1: now also U2.23 (DVDD), U2.45 (VREG_VOUT), U2.50 (DVDD)
- net +3V3: now also U2.1 (IOVDD), U2.10 (IOVDD), U2.22 (IOVDD), U2.26 (RUN), U2.33 (IOVDD), U2.42 (IOVDD), U2.43 (ADC_AVDD), U2.48 (USB_VDD), U2.49 (IOVDD), TP5.1
- net DEBUG1: now also U2.29 (GPIO18)
- net DEBUG2: now also U2.30 (GPIO19)
- net DEBUG3: now also U2.31 (GPIO20)
- net LED1: now also U2.2 (GPIO0); no longer U2.6 (GPIO4)
- net LED2: now also U2.3 (GPIO1); no longer U2.7 (GPIO5)
- net UART_RX: now also U2.28 (GPIO17), U5.1 (A); no longer U2.3 (GPIO1), U4.1 (A)
- net UART_RX_OUT: now also U5.4 (Y); no longer U4.4 (Y)
- net UART_TX: now also U2.27 (GPIO16), U4.1 (A); no longer U2.2 (GPIO0), U5.1 (A)
- net UART_TX_OUT: now also U4.4 (Y); no longer U5.4 (Y)
- net VBUS: now also TP4.1
- net YI: now also Y1.3; no longer Y1.2
- no-connect marks 7 -> 24
Other:
- note added: "Power Test Pads"
- moved on the sheet: U4, U5

Commit message: Add v1.1.1 schematic and PCB
Parts:
- R1: footprint Resistor_SMD:R_0603_1608Metric -> Resistor_SMD:R_0402_1005Metric
Connections:
- net +3V3: no longer D1.3 (VDD), D2.3 (VDD)
- net LED2: now also U2.15 (GPIO12); no longer U2.3 (GPIO1)
- net VBUS: now also D1.3 (VDD), D2.3 (VDD)
Changed lines of the file:
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@@
     (title "Expansion Card Template")
     (date "2022-12-28")
-    (rev "V1.1.1")
+    (rev "V1.1.3")
     (company "Framework")
     (comment 1 "This work is licensed under a Creative Commons Attribution 4.0 International License")
@@
   )
   (no_connect (at 173.99 58.42))
-  (no_connect (at 173.99 73.66))
   (no_connect (at 173.99 68.58))
   (no_connect (at 173.99 96.52))
@@
   (no_connect (at 173.99 71.12))
   (no_connect (at 173.99 114.3))
+  (no_connect (at 173.99 45.72))
   (no_connect (at 173.99 99.06))
   (no_connect (at 173.99 60.96))
@@
     (stroke (width 0) (type default) (color 0 0 0 0))
   )
-  (wire (pts (xy 173.99 45.72) (xy 185.42 45.72))
-    (stroke (width 0) (type default) (color 0 0 0 0))
-  )
   (wire (pts (xy 111.76 60.96) (xy 123.19 60.96))
     (stroke (width 0) (type default) (color 0 0 0 0))
@@
   )
   (wire (pts (xy 76.2 121.92) (xy 86.36 121.92))
+    (stroke (width 0) (type default) (color 0 0 0 0))
+  )
+  (wire (pts (xy 173.99 73.66) (xy 182.88 73.66))
     (stroke (width 0) (type default) (color 0 0 0 0))
   )
@@
     (effects (font (size 1.27 1.27)) (justify left bottom))
   )
+  (label "LED2" (at 182.88 73.66 0)
+    (effects (font (size 1.27 1.27)) (justify left bottom))
+  )
   (label "GND" (at 88.9 190.5 0)
     (effects (font (size 1.27 1.27)) (justify left bottom))
@@
   )
   (label "DEBUG1" (at 175.26 88.9 0)
-    (effects (font (size 1.27 1.27)) (justify left bottom))
-  )
-  (label "LED2" (at 185.42 45.72 0)
     (effects (font (size 1.27 1.27)) (justify left bottom))
   )
@@
       (effects (font (size 1.27 1.27)) (justify left))
     )
-    (property "Footprint" "Resistor_SMD:R_0603_1608Metric" (id 2) (at 67.31 40.64 0)
+    (property "Footprint" "Resistor_SMD:R_0402_1005Metric" (id 2) (at 67.31 40.64 0)
       (effects (font (size 1.27 1.27)) hide)
     )
@@
     (pin "3")
     (pin "4")
+  )
+  (symbol (lib_id "power:VBUS") (at 260.35 107.95 0) (unit 1)
+    (in_bom yes) (on_board yes)
+    (property "Reference" "#PWR0105" (id 0) (at 260.35 111.76 0)
+      (effects (font (size 1.27 1.27)) hide)
+    )
+    (property "Value" "VBUS" (id 1) (at 260.731 103.5558 0))
+    (property "Footprint" "" (id 2) (at 260.35 107.95 0)
+      (effects (font (size 1.27 1.27)) hide)
+    )
+    (property "Datasheet" "" (id 3) (at 260.35 107.95 0)
+      (effects (font (size 1.27 1.27)) hide)
+    )
+    (pin "1")
   )
   (symbol (lib_id "Memory_Flash:W25Q128JVS") (at 40.64 162.56 0) (unit 1)
@@
     (pin "1")
     (pin "2")
-  )
-  (symbol (lib_id "power:+3V3") (at 260.35 107.95 0) (unit 1)
-    (in_bom yes) (on_board yes)
-    (property "Reference" "#PWR018" (id 0) (at 260.35 111.76 0)
-      (effects (font (size 1.27 1.27)) hide)
-    )
-    (property "Value" "+3V3" (id 1) (at 260.35 104.14 0))
-    (property "Footprint" "" (id 2) (at 260.35 107.95 0)
-      (effects (font (size 1.27 1.27)) hide)
-    )
-    (property "Datasheet" "" (id 3) (at 260.35 107.95 0)
-      (effects (font (size 1.27 1.27)) hide)
-    )
-    (pin "1")
   )
   (symbol (lib_id "power:+3V3") (at 120.65 30.48 0) (unit 1)
@@
     (pin "5")
   )
-  (symbol (lib_id "power:+3V3") (at 260.35 138.43 0) (unit 1)
-    (in_bom yes) (on_board yes)
-    (property "Reference" "#PWR021" (id 0) (at 260.35 142.24 0)
-      (effects (font (size 1.27 1.27)) hide)
-    )
-    (property "Value" "+3V3" (id 1) (at 260.35 134.62 0))
-    (property "Footprint" "" (id 2) (at 260.35 138.43 0)
-      (effects (font (size 1.27 1.27)) hide)
-    )
-    (property "Datasheet" "" (id 3) (at 260.35 138.43 0)
-      (effects (font (size 1.27 1.27)) hide)
-    )
-    (pin "1")
-  )
   (symbol (lib_id "power:+3V3") (at 246.38 24.13 0) (unit 1)
     (in_bom yes) (on_board yes)
@@
     )
     (property "Datasheet" "" (id 3) (at 210.82 96.52 0)
+      (effects (font (size 1.27 1.27)) hide)
+    )
+    (pin "1")
+  )
+  (symbol (lib_id "power:VBUS") (at 260.35 138.43 0) (unit 1)
+    (in_bom yes) (on_board yes)
+    (property "Reference" "#PWR0104" (id 0) (at 260.35 142.24 0)
+      (effects (font (size 1.27 1.27)) hide)
+    )
+    (property "Value" "VBUS" (id 1) (at 260.731 134.0358 0))
+    (property "Footprint" "" (id 2) (at 260.35 138.43 0)
+      (effects (font (size 1.27 1.27)) hide)
+    )
+    (property "Datasheet" "" (id 3) (at 260.35 138.43 0)
       (effects (font (size 1.27 1.27)) hide)
     )
@@
       (reference "#PWR017") (unit 1) (value "GND") (footprint "")
     )
-    (path "/79862796-faa8-484b-9838-b3ec6449c310"
-      (reference "#PWR018") (unit 1) (value "+3V3") (footprint "")
-    )
     (path "/439b6ada-fc0d-4d82-9d6a-58af5754dac4"
       (reference "#PWR019") (unit 1) (value "GND") (footprint "")
@@
       (reference "#PWR020") (unit 1) (value "GND") (footprint "")
     )
-    (path "/b7d7229b-45ea-4543-8015-f45e69d4f20e"
-      (reference "#PWR021") (unit 1) (value "+3V3") (footprint "")
-    )
     (path "/91835499-ab6b-41ff-8c13-09a7992d39f3"
       (reference "#PWR022") (unit 1) (value "+3V3") (footprint "")
@@
       (reference "#PWR0103") (unit 1) (value "+3V3") (footprint "")
     )
+    (path "/d843b3a8-0d23-48cb-82e7-b09a3833d65a"
+      (reference "#PWR0104") (unit 1) (value "VBUS") (footprint "")
+    )
+    (path "/576aafda-7095-44c9-b38e-260762a778c0"
+      (reference "#PWR0105") (unit 1) (value "VBUS") (footprint "")
+    )
     (path "/00000000-0000-0000-0000-00005fd33d8e"
       (reference "C1") (unit 1) (value "10uF") (footprint "Capacitor_SMD:C_0805_2012Metric")
@@
     )
     (path "/00000000-0000-0000-0000-00005fd77c84"
-      (reference "R1") (unit 1) (value "5.1k") (footprint "Resistor_SMD:R_0603_1608Metric")
+      (reference "R1") (unit 1) (value "5.1k") (footprint "Resistor_SMD:R_0402_1005Metric")
     )
     (path "/fc9cffb7-904a-44c8-b4a4-cda1aab3e94b"
